File: projects/ESC/ESC.sch (EAGLE design)
At the start: 79 parts, among them J2 1755529, U1 STM32F405RGT6, U10 CSD88584Q5DCT, U11 CSD88584Q5DCT, U12 CSD88584Q5DCT, U13 CSD88584Q5DCT, U2 CSD88584Q5DCT, U3 CSD88584Q5DCT, U4 CSD88584Q5DCT, U5 CSD88584Q5DCT, U6 CSD88584Q5DCT, U7 CSD88584Q5DCT, U8 CSD88584Q5DCT, U9 CSD88584Q5DCT, Y1 ABLS2-4.096MHZ-D4Y-T

Commit message: VM'd 6-packs
Connections:
- removed net +12V: U10.VIN, U11.VIN, U12.VIN, U13.VIN, U5.VIN, U6.VIN, U7.VIN, U8.VIN, U9.VIN
- net VM_2: now also U5.VIN, U6.VIN, U7.VIN
- net VM_3: now also U10.VIN, U8.VIN, U9.VIN
- net VM_4: now also U11.VIN, U12.VIN, U13.VIN
Changed lines of the file:
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@@
 <part name="U6" library="VESC_SHIT" deviceset="CSD88584Q5DCT" device=""/>
 <part name="U7" library="VESC_SHIT" deviceset="CSD88584Q5DCT" device=""/>
-<part name="P+2" library="supply1" library_urn="urn:adsk.eagle:library:371" deviceset="+12V" device=""/>
 <part name="U8" library="VESC_SHIT" deviceset="CSD88584Q5DCT" device=""/>
 <part name="U9" library="VESC_SHIT" deviceset="CSD88584Q5DCT" device=""/>
 <part name="U10" library="VESC_SHIT" deviceset="CSD88584Q5DCT" device=""/>
-<part name="P+3" library="supply1" library_urn="urn:adsk.eagle:library:371" deviceset="+12V" device=""/>
 <part name="U11" library="VESC_SHIT" deviceset="CSD88584Q5DCT" device=""/>
 <part name="U12" library="VESC_SHIT" deviceset="CSD88584Q5DCT" device=""/>
 <part name="U13" library="VESC_SHIT" deviceset="CSD88584Q5DCT" device=""/>
-<part name="P+4" library="supply1" library_urn="urn:adsk.eagle:library:371" deviceset="+12V" device=""/>
 <part name="J2" library="VESC_SHIT" deviceset="1755529" device=""/>
 <part name="SV2" library="con-lsta" library_urn="urn:adsk.eagle:library:161" deviceset="FE05-1" device="" package3d_urn="urn:adsk.eagle:package:8190/1"/>
@@
 <attribute name="VALUE" x="68.3006" y="19.2786" size="2.0828" layer="96" ratio="6" rot="SR0"/>
 </instance>
-<instance part="P+2" gate="1" x="0" y="35.56" smashed="yes">
-<attribute name="VALUE" x="-2.54" y="30.48" size="1.778" layer="96" rot="R90"/>
-</instance>
 </instances>
 <busses>
 </busses>
 <nets>
-<net name="+12V" class="0">
-<segment>
-<pinref part="P+2" gate="1" pin="+12V"/>
-<wire x1="0" y1="33.02" x2="-45.72" y2="33.02" width="0.1524" layer="91"/>
-<wire x1="-45.72" y1="33.02" x2="-45.72" y2="15.24" width="0.1524" layer="91"/>
-<pinref part="U6" gate="A" pin="VIN"/>
-<wire x1="-45.72" y1="15.24" x2="-55.88" y2="15.24" width="0.1524" layer="91"/>
-<wire x1="0" y1="33.02" x2="33.02" y2="33.02" width="0.1524" layer="91"/>
-<junction x="0" y="33.02"/>
-<wire x1="33.02" y1="33.02" x2="33.02" y2="15.24" width="0.1524" layer="91"/>
-<pinref part="U5" gate="A" pin="VIN"/>
-<wire x1="33.02" y1="15.24" x2="17.78" y2="15.24" width="0.1524" layer="91"/>
-<wire x1="33.02" y1="33.02" x2="99.06" y2="33.02" width="0.1524" layer="91"/>
-<junction x="33.02" y="33.02"/>
-<wire x1="99.06" y1="33.02" x2="99.06" y2="12.7" width="0.1524" layer="91"/>
-<pinref part="U7" gate="A" pin="VIN"/>
-<wire x1="99.06" y1="12.7" x2="91.44" y2="12.7" width="0.1524" layer="91"/>
-</segment>
-</net>
 <net name="GHA_2" class="0">
 <segment>
@@
 </segment>
 </net>
+<net name="VM_2" class="0">
+<segment>
+<wire x1="33.02" y1="33.02" x2="-45.72" y2="33.02" width="0.1524" layer="91"/>
+<wire x1="-45.72" y1="33.02" x2="-45.72" y2="15.24" width="0.1524" layer="91"/>
+<pinref part="U6" gate="A" pin="VIN"/>
+<wire x1="-45.72" y1="15.24" x2="-55.88" y2="15.24" width="0.1524" layer="91"/>
+<wire x1="33.02" y1="33.02" x2="33.02" y2="15.24" width="0.1524" layer="91"/>
+<pinref part="U5" gate="A" pin="VIN"/>
+<wire x1="33.02" y1="15.24" x2="17.78" y2="15.24" width="0.1524" layer="91"/>
+<wire x1="33.02" y1="33.02" x2="99.06" y2="33.02" width="0.1524" layer="91"/>
+<junction x="33.02" y="33.02"/>
+<wire x1="99.06" y1="33.02" x2="99.06" y2="12.7" width="0.1524" layer="91"/>
+<pinref part="U7" gate="A" pin="VIN"/>
+<wire x1="99.06" y1="12.7" x2="91.44" y2="12.7" width="0.1524" layer="91"/>
+<label x="33.02" y="33.02" size="1.778" layer="95"/>
+</segment>
+</net>
 </nets>
 </sheet>
@@
 <attribute name="VALUE" x="68.3006" y="19.2786" size="2.0828" layer="96" ratio="6" rot="SR0"/>
 </instance>
-<instance part="P+3" gate="1" x="0" y="35.56" smashed="yes">
-<attribute name="VALUE" x="-2.54" y="30.48" size="1.778" layer="96" rot="R90"/>
-</instance>
 </instances>
 <busses>
 </busses>
 <nets>
-<net name="+12V" class="0">
-<segment>
-<pinref part="P+3" gate="1" pin="+12V"/>
-<wire x1="0" y1="33.02" x2="-45.72" y2="33.02" width="0.1524" layer="91"/>
-<wire x1="-45.72" y1="33.02" x2="-45.72" y2="15.24" width="0.1524" layer="91"/>
-<pinref part="U9" gate="A" pin="VIN"/>
-<wire x1="-45.72" y1="15.24" x2="-55.88" y2="15.24" width="0.1524" layer="91"/>
-<wire x1="0" y1="33.02" x2="33.02" y2="33.02" width="0.1524" layer="91"/>
-<junction x="0" y="33.02"/>
-<wire x1="33.02" y1="33.02" x2="33.02" y2="15.24" width="0.1524" layer="91"/>
-<pinref part="U8" gate="A" pin="VIN"/>
-<wire x1="33.02" y1="15.24" x2="17.78" y2="15.24" width="0.1524" layer="91"/>
-<wire x1="33.02" y1="33.02" x2="99.06" y2="33.02" width="0.1524" layer="91"/>
-<junction x="33.02" y="33.02"/>
-<wire x1="99.06" y1="33.02" x2="99.06" y2="12.7" width="0.1524" layer="91"/>
-<pinref part="U10" gate="A" pin="VIN"/>
-<wire x1="99.06" y1="12.7" x2="91.44" y2="12.7" width="0.1524" layer="91"/>
-</segment>
-</net>
 <net name="GHA_3" class="0">
 <segment>
@@
 </segment>
 </net>
+<net name="VM_3" class="0">
+<segment>
+<wire x1="33.02" y1="33.02" x2="-45.72" y2="33.02" width="0.1524" layer="91"/>
+<wire x1="-45.72" y1="33.02" x2="-45.72" y2="15.24" width="0.1524" layer="91"/>
+<pinref part="U9" gate="A" pin="VIN"/>
+<wire x1="-45.72" y1="15.24" x2="-55.88" y2="15.24" width="0.1524" layer="91"/>
+<wire x1="33.02" y1="33.02" x2="33.02" y2="15.24" width="0.1524" layer="91"/>
+<pinref part="U8" gate="A" pin="VIN"/>
+<wire x1="33.02" y1="15.24" x2="17.78" y2="15.24" width="0.1524" layer="91"/>
+<wire x1="33.02" y1="33.02" x2="99.06" y2="33.02" width="0.1524" layer="91"/>
+<junction x="33.02" y="33.02"/>
+<wire x1="99.06" y1="33.02" x2="99.06" y2="12.7" width="0.1524" layer="91"/>
+<pinref part="U10" gate="A" pin="VIN"/>
+<wire x1="99.06" y1="12.7" x2="91.44" y2="12.7" width="0.1524" layer="91"/>
+<label x="33.02" y="33.02" size="1.778" layer="95"/>
+</segment>
+</net>
 </nets>
 </sheet>
@@
 <attribute name="VALUE" x="68.3006" y="19.2786" size="2.0828" layer="96" ratio="6" rot="SR0"/>
 </instance>
-<instance part="P+4" gate="1" x="0" y="35.56" smashed="yes">
-<attribute name="VALUE" x="-2.54" y="30.48" size="1.778" layer="96" rot="R90"/>
-</instance>
 </instances>
 <busses>
 </busses>
 <nets>
-<net name="+12V" class="0">
-<segment>
-<pinref part="P+4" gate="1" pin="+12V"/>
-<wire x1="0" y1="33.02" x2="-45.72" y2="33.02" width="0.1524" layer="91"/>
-<wire x1="-45.72" y1="33.02" x2="-45.72" y2="15.24" width="0.1524" layer="91"/>
-<pinref part="U12" gate="A" pin="VIN"/>
-<wire x1="-45.72" y1="15.24" x2="-55.88" y2="15.24" width="0.1524" layer="91"/>
-<wire x1="0" y1="33.02" x2="33.02" y2="33.02" width="0.1524" layer="91"/>
-<junction x="0" y="33.02"/>
-<wire x1="33.02" y1="33.02" x2="33.02" y2="15.24" width="0.1524" layer="91"/>
-<pinref part="U11" gate="A" pin="VIN"/>
-<wire x1="33.02" y1="15.24" x2="17.78" y2="15.24" width="0.1524" layer="91"/>
-<wire x1="33.02" y1="33.02" x2="99.06" y2="33.02" width="0.1524" layer="91"/>
-<junction x="33.02" y="33.02"/>
-<wire x1="99.06" y1="33.02" x2="99.06" y2="12.7" width="0.1524" layer="91"/>
-<pinref part="U13" gate="A" pin="VIN"/>
-<wire x1="99.06" y1="12.7" x2="91.44" y2="12.7" width="0.1524" layer="91"/>
-</segment>
-</net>
 <net name="GHA_4" class="0">
 <segment>
@@
 </segment>
 </net>
+<net name="VM_4" class="0">
+<segment>
+<wire x1="33.02" y1="33.02" x2="-45.72" y2="33.02" width="0.1524" layer="91"/>
+<wire x1="-45.72" y1="33.02" x2="-45.72" y2="15.24" width="0.1524" layer="91"/>
+<pinref part="U12" gate="A" pin="VIN"/>
+<wire x1="-45.72" y1="15.24" x2="-55.88" y2="15.24" width="0.1524" layer="91"/>
+<wire x1="33.02" y1="33.02" x2="33.02" y2="15.24" width="0.1524" layer="91"/>
+<pinref part="U11" gate="A" pin="VIN"/>
+<wire x1="33.02" y1="15.24" x2="17.78" y2="15.24" width="0.1524" layer="91"/>
+<wire x1="33.02" y1="33.02" x2="99.06" y2="33.02" width="0.1524" layer="91"/>
+<junction x="33.02" y="33.02"/>
+<wire x1="99.06" y1="33.02" x2="99.06" y2="12.7" width="0.1524" layer="91"/>
+<pinref part="U13" gate="A" pin="VIN"/>
+<wire x1="99.06" y1="12.7" x2="91.44" y2="12.7" width="0.1524" layer="91"/>
+<label x="33.02" y="33.02" size="1.778" layer="95"/>
+</segment>
+</net>
