File: projects/ESC/ESC.sch (EAGLE design)
At the start: 91 parts, among them J1 1755529, J2 1755529, J3 1755529, J4 1755529, U1 STM32F405RGT6, U10 CSD88584Q5DCT, U11 CSD88584Q5DCT, U12 CSD88584Q5DCT, U13 CSD88584Q5DCT, U2 CSD88584Q5DCT, U3 CSD88584Q5DCT, U4 CSD88584Q5DCT, U5 CSD88584Q5DCT, U6 CSD88584Q5DCT, U7 CSD88584Q5DCT, U8 CSD88584Q5DCT, U9 CSD88584Q5DCT, Y1 ECS-80-S-4X

Commit message: pre-meeting changes
Connections:
- removed net 3V3: U$5G$1.1, U$5G$1.10, U$5G$1.11, U$5G$1.12, U$5G$1.13, U$5G$1.14, U$5G$1.15, U$5G$1.16, U$5G$1.17, U$5G$1.18, U$5G$1.19, U$5G$1.2, U$5G$1.20, U$5G$1.21, U$5G$1.22, U$5G$1.23, U$5G$1.24, U$5G$1.3, U$5G$1.4, U$5G$1.5, U$5G$1.6, U$5G$1.7, U$5G$1.8, U$5G$1.9, U1.VBAT, U1.VDDA, U1.VDD_1, U1.VDD_2, U1.VDD_3, U1.VDD_4
- net +3V3: now also U$5G$1.1, U$5G$1.10, U$5G$1.11, U$5G$1.12, U$5G$1.13, U$5G$1.14, U$5G$1.15, U$5G$1.16, U$5G$1.17, U$5G$1.18, U$5G$1.19, U$5G$1.2, U$5G$1.20, U$5G$1.21, U$5G$1.22, U$5G$1.23, U$5G$1.24, U$5G$1.3, U$5G$1.4, U$5G$1.5, U$5G$1.6, U$5G$1.7, U$5G$1.8, U$5G$1.9, U1.VBAT, U1.VDDA, U1.VDD_1, U1.VDD_2, U1.VDD_3, U1.VDD_4
- net EN_3: now also U1.PB3; no longer U1.PD2
- net FAULT_3: now also U1.PD2; no longer U1.PB3
- net INHA_3: now also U1.PB4; no longer U1.PC12
- net INHA_4: now also U1.PA15; no longer U1.PB7
- net INHB_3: now also U1.PB5; no longer U1.PC11
- net INHB_4: now also U1.PC10; no longer U1.PB6
- net INHC_3: now also U1.PB7; no longer U1.PC10
- net INHC_4: now also U1.PC12; no longer U1.PB5
- net INL_3: now also U1.PB6; no longer U1.PA15
- net INL_4: now also U1.PC11; no longer U1.PB4

Commit message: RIPUP MY LIFE
Parts:
- removed U$7: SAMTEC, VESC_SHIT:SAMTEC
- U$5: value SAMTEC -> ESC2BACKPLANE; device VESC_SHIT:SAMTEC -> ESC_to_Backplane_Connectors:ESC2BACKPLANE
Connections:
- removed net 12V: U$5G$2.1, U$5G$2.10, U$5G$2.11, U$5G$2.12, U$5G$2.13, U$5G$2.14, U$5G$2.15, U$5G$2.16, U$5G$2.17, U$5G$2.18, U$5G$2.19, U$5G$2.2, U$5G$2.20, U$5G$2.21, U$5G$2.22, U$5G$2.23, U$5G$2.24, U$5G$2.25, U$5G$2.26, U$5G$2.27, U$5G$2.28, U$5G$2.29, U$5G$2.3, U$5G$2.30, U$5G$2.31, U$5G$2.32, U$5G$2.4, U$5G$2.5, U$5G$2.6, U$5G$2.7, U$5G$2.8, U$5G$2.9
- net +3V3: no longer U$5G$1.1, U$5G$1.10, U$5G$1.11, U$5G$1.12, U$5G$1.13, U$5G$1.14, U$5G$1.15, U$5G$1.16, U$5G$1.17, U$5G$1.18, U$5G$1.19, U$5G$1.2, U$5G$1.20, U$5G$1.21, U$5G$1.22, U$5G$1.23, U$5G$1.24, U$5G$1.3, U$5G$1.4, U$5G$1.5, U$5G$1.6, U$5G$1.7, U$5G$1.8, U$5G$1.9
- net CAN_H: no longer U$7G$1.24
- net CAN_L: no longer U$7G$1.23
- net GND: no longer U$7G$2.1, U$7G$2.10, U$7G$2.11, U$7G$2.12, U$7G$2.13, U$7G$2.14, U$7G$2.15, U$7G$2.16, U$7G$2.17, U$7G$2.18, U$7G$2.19, U$7G$2.2, U$7G$2.20, U$7G$2.21, U$7G$2.22, U$7G$2.23, U$7G$2.24, U$7G$2.25, U$7G$2.26, U$7G$2.27, U$7G$2.28, U$7G$2.29, U$7G$2.3, U$7G$2.30, U$7G$2.31, U$7G$2.32, U$7G$2.4, U$7G$2.5, U$7G$2.6, U$7G$2.7, U$7G$2.8, U$7G$2.9

Commit message: making some changes
Parts:
- added C6: 0.1uF, SparkFun-Capacitors:0.1UF-0603-25V-(+80/-20%)
- added R6: 1.5k, SparkFun-Resistors:1.5KOHM-0603-1/10W-1%
- added U14: SN74CBTLV3257PWR, SN74CBTLV3257PWR:SN74CBTLV3257PWR
Connections:
- new net +12V: U$5G$1.P$10, U$5G$1.P$11, U$5G$1.P$12, U$5G$1.P$13, U$5G$1.P$23, U$5G$1.P$24, U$5G$1.P$25, U$5G$1.P$26, U$5G$1.P$27, U$5G$1.P$9, U$5G$2.P$A, U$5G$2.P$B, U$5G$2.P$C, U$5G$2.P$D, U$5G$2.P$E, U$5G$2.P$O, U$5G$2.P$P, U$5G$2.P$Q, U$5G$2.P$R, U$5G$2.P$S
- new net N$10: R6.1, U14.OE
- new net NRST_IN: U14.3A
- new net PROG_SEL: U$5G$1.P$5
- new net S: U$6.S, U14.S
- new net SWCLK_IN: U14.1A
- new net SWDIO_IN: U14.2A
- net +3V3: now also C6.1, R6.2, U$5G$2.P$G, U$5G$2.P$H, U$5G$2.P$U, U$5G$2.P$V, U14.VCC
- net CAN_H: now also U$5G$1.P$6
- net CAN_L: now also U$5G$1.P$7
- net GND: now also C6.2, U$5G$1.P$1, U$5G$1.P$15, U$5G$1.P$16, U$5G$1.P$17, U$5G$1.P$18, U$5G$1.P$2, U$5G$1.P$3, U$5G$1.P$4, U$5G$2.P$AA, U$5G$2.P$BB, U$5G$2.P$J, U$5G$2.P$K, U$5G$2.P$L, U$5G$2.P$M, U$5G$2.P$N, U$5G$2.P$X, U$5G$2.P$Y, U$5G$2.P$Z, U14.GND
- net NRST: now also U14.3B1
- net SWCLK: now also U14.1B1
- net SWDIO: now also U14.2B1

Commit message: All 4 drive ckts complete
Added and implemented design block across all 4 motors.
Parts:
- removed C18: 47nF, SparkFun-Capacitors:47NF-0603-25V-5%
- removed R13: 47k, rcl:R-US_R0603
- removed R14, R15, R16: (no value), rcl:R-US_R0603
- removed U$1: DRV8320H, VESC_SHIT:DRV8320H
- removed U5, U6, U7: CSD88584Q5DCT, VESC_SHIT:CSD88584Q5DCT
- added C36: 1.0uF, SparkFun-Capacitors:1.0UF-0603-16V-10%
- added R30, R31, R32, R33: (no value), rcl:R-US_R0603
- added U$7: DRV8320H, VESC_SHIT:DRV8320H
- added U15, U16, U17: CSD88584Q5DCT, VESC_SHIT:CSD88584Q5DCT
- C19, C23, C27: value 1.0uF -> 47nF; device SparkFun-Capacitors:1.0UF-0603-16V-10% -> SparkFun-Capacitors:47NF-0603-25V-5%
- C20, C24, C28: value 0.1uF -> 1.0uF; device SparkFun-Capacitors:0.1UF-0603-25V-(+80/-20%) -> SparkFun-Capacitors:1.0UF-0603-16V-10%
- C21, C25, C29: value 1.0uF -> 0.1uF; device SparkFun-Capacitors:1.0UF-0603-16V-10% -> SparkFun-Capacitors:0.1UF-0603-25V-(+80/-20%)
- C22, C26: value 47nF -> 1.0uF; device SparkFun-Capacitors:47NF-0603-25V-5% -> SparkFun-Capacitors:1.0UF-0603-16V-10%
- R17, R22, R27: value (none) -> 47k
- R18, R23: value 47k -> (none)
Connections:
- removed net IDRIVE: R19.1, R20.2, U$1G$1.IDRIVE
- removed net N$25: C18.2, U$3G$1.CPL
- removed net N$31: C22.1, U$1G$1.CPH
- removed net N$40: C29.1, U$4G$2.VCP
- removed net N$41: C26.1, U$4G$1.CPH
- removed net N$42: C26.2, U$4G$1.CPL
- removed net N$43: R24.1, R25.2, U$4G$1.IDRIVE
- removed net N$44: R23.2, U$4G$1.MODE
- removed net N$45: R26.1, R27.2, U$4G$1.VDS
- removed net VDS: R21.1, R22.2, U$1G$1.VDS
- new net N$11: R17.2, U$3G$1.MODE
- new net N$12: R22.2, U$4G$1.MODE
- new net N$13: R27.2, U$7G$1.MODE
- new net N$21: C22.1, U$3G$2.VCP
- new net N$22: C19.1, U$3G$1.CPH
- new net N$29: C23.2, U$4G$1.CPL
- new net N$33: C36.1, U$7G$2.VCP
- new net N$36: C27.2, U$7G$1.CPL
- new net N$37: R30.1, R31.2, U$7G$1.IDRIVE
- new net N$39: R32.1, R33.2, U$7G$1.VDS
- net DVDD_2: now also C20.1, R18.2, R20.2, U$3G$2.DVDD; no longer C23.1, R19.2, R21.2, U$1G$2.DVDD
- net DVDD_3: now also C24.1, R23.2, R25.2, U$4G$2.DVDD; no longer C19.1, R14.2, R16.2, U$3G$2.DVDD
- net DVDD_4: now also C28.1, R30.2, R32.2, U$7G$2.DVDD; no longer C27.1, R24.2, R26.2, U$4G$2.DVDD
- net EN_2: now also U$3G$1.ENABLE; no longer U$1G$1.ENABLE
- net EN_3: now also U$4G$1.ENABLE; no longer U$3G$1.ENABLE
- net EN_4: now also U$7G$1.ENABLE; no longer U$4G$1.ENABLE
- net FAULT_2: now also U$3G$1.FAULT_N; no longer U$1G$1.FAULT_N
- net FAULT_3: now also U$4G$1.FAULT_N; no longer U$3G$1.FAULT_N
- net FAULT_4: now also U$7G$1.FAULT_N; no longer U$4G$1.FAULT_N
- net GHA_2: now also U$3G$1.GHA, U9.GH; no longer U$1G$1.GHA, U6.GH
- net GHA_3: now also U$4G$1.GHA, U12.GH; no longer U$3G$1.GHA, U9.GH
- net GHA_4: now also U$7G$1.GHA, U16.GH; no longer U$4G$1.GHA, U12.GH
- net GHB_2: now also U$3G$1.GHB, U10.GH; no longer U$1G$1.GHB, U5.GH
- net GHB_3: now also U$4G$1.GHB, U13.GH; no longer U$3G$1.GHB, U8.GH
- net GHB_4: now also U$7G$1.GHB, U17.GH; no longer U$4G$1.GHB, U11.GH
- net GHC_2: now also U$3G$1.GHC, U8.GH; no longer U$1G$1.GHC, U7.GH
- net GHC_3: now also U$4G$1.GHC, U11.GH; no longer U$3G$1.GHC, U10.GH
- net GHC_4: now also U$7G$1.GHC, U15.GH; no longer U$4G$1.GHC, U13.GH
- net GLA_2: now also U$3G$1.GLA, U9.GL; no longer U$1G$1.GLA, U6.GL
- net GLA_3: now also U$4G$1.GLA, U12.GL; no longer U$3G$1.GLA, U9.GL
- net GLA_4: now also U$7G$1.GLA, U16.GL; no longer U$4G$1.GLA, U12.GL
- net GLB_2: now also U$3G$1.GLB, U10.GL; no longer U$1G$1.GLB, U5.GL
- net GLB_3: now also U$4G$1.GLB, U13.GL; no longer U$3G$1.GLB, U8.GL
- net GLB_4: now also U$7G$1.GLB, U17.GL; no longer U$4G$1.GLB, U11.GL
- net GLC_2: now also U$3G$1.GLC, U8.GL; no longer U$1G$1.GLC, U7.GL
- net GLC_3: now also U$4G$1.GLC, U11.GL; no longer U$3G$1.GLC, U10.GL
- net GLC_4: now also U$7G$1.GLC, U15.GL; no longer U$4G$1.GLC, U13.GL
- net GND: now also C21.2, C25.2, C29.2, R19.1, R21.1, R24.1, R26.1, R31.1, R33.1, U$7G$2.AGND, U$7G$2.PAD, U$7G$2.PGND; no longer C19.2, C23.2, C27.2, R13.1, R15.1, R18.1, R20.1, R23.1, R25.1, U$1G$2.AGND, U$1G$2.PAD, U$1G$2.PGND
- net INHA_2: now also U$3G$1.INHA; no longer U$1G$1.INHA
- net INHA_3: now also U$4G$1.INHA; no longer U$3G$1.INHA
- net INHA_4: now also U$7G$1.INHA; no longer U$4G$1.INHA
- net INHB_2: now also U$3G$1.INHB; no longer U$1G$1.INHB
- net INHB_3: now also U$4G$1.INHB; no longer U$3G$1.INHB
- net INHB_4: now also U$7G$1.INHB; no longer U$4G$1.INHB
- net INHC_2: now also U$3G$1.INHC; no longer U$1G$1.INHC
- net INHC_3: now also U$4G$1.INHC; no longer U$3G$1.INHC
- net INHC_4: now also U$7G$1.INHC; no longer U$4G$1.INHC
- net INL_2: now also U$3G$1.INLA, U$3G$1.INLB, U$3G$1.INLC; no longer U$1G$1.INLA, U$1G$1.INLB, U$1G$1.INLC
- net INL_3: now also U$4G$1.INLA, U$4G$1.INLB, U$4G$1.INLC; no longer U$3G$1.INLA, U$3G$1.INLB, U$3G$1.INLC
- net INL_4: now also U$7G$1.INLA, U$7G$1.INLB, U$7G$1.INLC; no longer U$4G$1.INLA, U$4G$1.INLB, U$4G$1.INLC
- net N$23: now also C19.2, U$3G$1.CPL; no longer C21.1, U$3G$2.VCP
- net N$24: now also R18.1, R19.2, U$3G$1.IDRIVE; no longer C18.1, U$3G$1.CPH
- net N$26: now also R20.1, R21.2, U$3G$1.VDS; no longer R14.1, R15.2, U$3G$1.IDRIVE
- net N$27: now also C26.1, U$4G$2.VCP; no longer R13.2, U$3G$1.MODE
- net N$28: now also C23.1, U$4G$1.CPH; no longer R16.1, R17.2, U$3G$1.VDS
- net N$30: now also R23.1, R24.2, U$4G$1.IDRIVE; no longer C25.1, U$1G$2.VCP
- net N$32: now also R25.1, R26.2, U$4G$1.VDS; no longer C22.2, U$1G$1.CPL
- net N$35: now also C27.1, U$7G$1.CPH; no longer R18.2, U$1G$1.MODE
- net PHASE_A2: now also U9.VSW, U9.VSW_2, U9.VSW_3, U9.VSW_4, U9.VSW_5, U9.VSW_6, U9.VSW_7, U9.VSW_8, U9.VSW_9; no longer U6.VSW, U6.VSW_2, U6.VSW_3, U6.VSW_4, U6.VSW_5, U6.VSW_6, U6.VSW_7, U6.VSW_8, U6.VSW_9
- net PHASE_A3: now also U12.VSW, U12.VSW_2, U12.VSW_3, U12.VSW_4, U12.VSW_5, U12.VSW_6, U12.VSW_7, U12.VSW_8, U12.VSW_9; no longer U9.VSW, U9.VSW_2, U9.VSW_3, U9.VSW_4, U9.VSW_5, U9.VSW_6, U9.VSW_7, U9.VSW_8, U9.VSW_9
- net PHASE_A4: now also U16.VSW, U16.VSW_2, U16.VSW_3, U16.VSW_4, U16.VSW_5, U16.VSW_6, U16.VSW_7, U16.VSW_8, U16.VSW_9; no longer U12.VSW, U12.VSW_2, U12.VSW_3, U12.VSW_4, U12.VSW_5, U12.VSW_6, U12.VSW_7, U12.VSW_8, U12.VSW_9
- net PHASE_B2: now also U10.VSW, U10.VSW_2, U10.VSW_3, U10.VSW_4, U10.VSW_5, U10.VSW_6, U10.VSW_7, U10.VSW_8, U10.VSW_9; no longer U5.VSW, U5.VSW_2, U5.VSW_3, U5.VSW_4, U5.VSW_5, U5.VSW_6, U5.VSW_7, U5.VSW_8, U5.VSW_9
- net PHASE_B3: now also U13.VSW, U13.VSW_2, U13.VSW_3, U13.VSW_4, U13.VSW_5, U13.VSW_6, U13.VSW_7, U13.VSW_8, U13.VSW_9; no longer U8.VSW, U8.VSW_2, U8.VSW_3, U8.VSW_4, U8.VSW_5, U8.VSW_6, U8.VSW_7, U8.VSW_8, U8.VSW_9
- net PHASE_B4: now also U17.VSW, U17.VSW_2, U17.VSW_3, U17.VSW_4, U17.VSW_5, U17.VSW_6, U17.VSW_7, U17.VSW_8, U17.VSW_9; no longer U11.VSW, U11.VSW_2, U11.VSW_3, U11.VSW_4, U11.VSW_5, U11.VSW_6, U11.VSW_7, U11.VSW_8, U11.VSW_9
- net PHASE_C2: now also U8.VSW, U8.VSW_2, U8.VSW_3, U8.VSW_4, U8.VSW_5, U8.VSW_6, U8.VSW_7, U8.VSW_8, U8.VSW_9; no longer U7.VSW, U7.VSW_2, U7.VSW_3, U7.VSW_4, U7.VSW_5, U7.VSW_6, U7.VSW_7, U7.VSW_8, U7.VSW_9
- net PHASE_C3: now also U11.VSW, U11.VSW_2, U11.VSW_3, U11.VSW_4, U11.VSW_5, U11.VSW_6, U11.VSW_7, U11.VSW_8, U11.VSW_9; no longer U10.VSW, U10.VSW_2, U10.VSW_3, U10.VSW_4, U10.VSW_5, U10.VSW_6, U10.VSW_7, U10.VSW_8, U10.VSW_9
- net PHASE_C4: now also U15.VSW, U15.VSW_2, U15.VSW_3, U15.VSW_4, U15.VSW_5, U15.VSW_6, U15.VSW_7, U15.VSW_8, U15.VSW_9; no longer U13.VSW, U13.VSW_2, U13.VSW_3, U13.VSW_4, U13.VSW_5, U13.VSW_6, U13.VSW_7, U13.VSW_8, U13.VSW_9
- net SHA_2: now also U$3G$1.SHA, U9.SH; no longer U$1G$1.SHA, U6.SH
- net SHA_3: now also U$4G$1.SHA, U12.SH; no longer U$3G$1.SHA, U9.SH
- net SHA_4: now also U$7G$1.SHA, U16.SH; no longer U$4G$1.SHA, U12.SH
- net SHB_2: now also U$3G$1.SHB, U10.SH; no longer U$1G$1.SHB, U5.SH
- net SHB_3: now also U$4G$1.SHB, U13.SH; no longer U$3G$1.SHB, U8.SH
- net SHB_4: now also U$7G$1.SHB, U17.SH; no longer U$4G$1.SHB, U11.SH
- net SHC_2: now also U$3G$1.SHC, U8.SH; no longer U$1G$1.SHC, U7.SH
- net SHC_3: now also U$4G$1.SHC, U11.SH; no longer U$3G$1.SHC, U10.SH
- net SHC_4: now also U$7G$1.SHC, U15.SH; no longer U$4G$1.SHC, U13.SH
- net SLA_2: now also U$3G$1.SLA, U9.PGND, U9.PGND_2, U9.PGND_3, U9.PGND_4, U9.PGND_5, U9.PGND_6, U9.PGND_7, U9.PGND_8, U9.PGND_9; no longer U$1G$1.SLA, U6.PGND, U6.PGND_2, U6.PGND_3, U6.PGND_4, U6.PGND_5, U6.PGND_6, U6.PGND_7, U6.PGND_8, U6.PGND_9
- net SLA_3: now also U$4G$1.SLA, U12.PGND, U12.PGND_2, U12.PGND_3, U12.PGND_4, U12.PGND_5, U12.PGND_6, U12.PGND_7, U12.PGND_8, U12.PGND_9; no longer U$3G$1.SLA, U9.PGND, U9.PGND_2, U9.PGND_3, U9.PGND_4, U9.PGND_5, U9.PGND_6, U9.PGND_7, U9.PGND_8, U9.PGND_9
- net SLA_4: now also U$7G$1.SLA, U16.PGND, U16.PGND_2, U16.PGND_3, U16.PGND_4, U16.PGND_5, U16.PGND_6, U16.PGND_7, U16.PGND_8, U16.PGND_9; no longer U$4G$1.SLA, U12.PGND, U12.PGND_2, U12.PGND_3, U12.PGND_4, U12.PGND_5, U12.PGND_6, U12.PGND_7, U12.PGND_8, U12.PGND_9
- net SLB_2: now also U$3G$1.SLB, U10.PGND, U10.PGND_2, U10.PGND_3, U10.PGND_4, U10.PGND_5, U10.PGND_6, U10.PGND_7, U10.PGND_8, U10.PGND_9; no longer U$1G$1.SLB, U5.PGND, U5.PGND_2, U5.PGND_3, U5.PGND_4, U5.PGND_5, U5.PGND_6, U5.PGND_7, U5.PGND_8, U5.PGND_9
- net SLB_3: now also U$4G$1.SLB, U13.PGND, U13.PGND_2, U13.PGND_3, U13.PGND_4, U13.PGND_5, U13.PGND_6, U13.PGND_7, U13.PGND_8, U13.PGND_9; no longer U$3G$1.SLB, U8.PGND, U8.PGND_2, U8.PGND_3, U8.PGND_4, U8.PGND_5, U8.PGND_6, U8.PGND_7, U8.PGND_8, U8.PGND_9
- net SLB_4: now also U$7G$1.SLB, U17.PGND, U17.PGND_2, U17.PGND_3, U17.PGND_4, U17.PGND_5, U17.PGND_6, U17.PGND_7, U17.PGND_8, U17.PGND_9; no longer U$4G$1.SLB, U11.PGND, U11.PGND_2, U11.PGND_3, U11.PGND_4, U11.PGND_5, U11.PGND_6, U11.PGND_7, U11.PGND_8, U11.PGND_9
- net SLC_2: now also U$3G$1.SLC, U8.PGND, U8.PGND_2, U8.PGND_3, U8.PGND_4, U8.PGND_5, U8.PGND_6, U8.PGND_7, U8.PGND_8, U8.PGND_9; no longer U$1G$1.SLC, U7.PGND, U7.PGND_2, U7.PGND_3, U7.PGND_4, U7.PGND_5, U7.PGND_6, U7.PGND_7, U7.PGND_8, U7.PGND_9
- net SLC_3: now also U$4G$1.SLC, U11.PGND, U11.PGND_2, U11.PGND_3, U11.PGND_4, U11.PGND_5, U11.PGND_6, U11.PGND_7, U11.PGND_8, U11.PGND_9; no longer U$3G$1.SLC, U10.PGND, U10.PGND_2, U10.PGND_3, U10.PGND_4, U10.PGND_5, U10.PGND_6, U10.PGND_7, U10.PGND_8, U10.PGND_9
- net SLC_4: now also U$7G$1.SLC, U15.PGND, U15.PGND_2, U15.PGND_3, U15.PGND_4, U15.PGND_5, U15.PGND_6, U15.PGND_7, U15.PGND_8, U15.PGND_9; no longer U$4G$1.SLC, U13.PGND, U13.PGND_2, U13.PGND_3, U13.PGND_4, U13.PGND_5, U13.PGND_6, U13.PGND_7, U13.PGND_8, U13.PGND_9
- net VM_2: now also C21.1, C22.2, U$3G$1.VDRAIN, U$3G$2.VM, U10.VIN, U8.VIN, U9.VIN; no longer C24.1, C25.2, U$1G$1.VDRAIN, U$1G$2.VM, U5.VIN, U6.VIN, U7.VIN
- net VM_3: now also C25.1, C26.2, U$4G$1.VDRAIN, U$4G$2.VM, U11.VIN, U12.VIN, U13.VIN; no longer C20.1, C21.2, U$3G$1.VDRAIN, U$3G$2.VM, U10.VIN, U8.VIN, U9.VIN
- net VM_4: now also C29.1, C36.2, U$7G$1.VDRAIN, U$7G$2.VM, U15.VIN, U16.VIN, U17.VIN; no longer C28.1, C29.2, U$4G$1.VDRAIN, U$4G$2.VM, U11.VIN, U12.VIN, U13.VIN
