File: projects/Test/test.brd (EAGLE design)
At the start: 63.5 x 24.1 mm, 47 parts, among them J2 1755529, U1 STM32F405RGT6, U2 CSD88584Q5DCT, U3 CSD88584Q5DCT, U4 CSD88584Q5DCT, Y1 ECS-80-S-4X

Commit message: stuff for jonah to drc
Parts:
- moved U2 0.26 mm to (14.8, 5.61)
Routing:
- net 12V: track 49.6 -> 110.9 mm
- net INL_1: track 8.58 -> 12.1 mm
- net GND: track 10.4 -> 12.8 mm, vias 2 -> 1
- net N$7: track 4.46 -> 5.61 mm
- net 3V3: track 69.3 -> 70.4 mm
- net SLB_1: track 23.1 -> 22.3 mm
- net FAULT_1: track 23.0 -> 23.5 mm

Commit message: some work on the test
Parts:
- moved R9 3.56 mm to (21.4, 3.20), turned to 180 degrees
- moved R8 3.18 mm to (24.0, 4.01), turned to 270 degrees
- moved R11 2.31 mm to (24.8, 3.28), flipped to the bottom, turned to 0 degrees
- moved R10 1.60 mm to (26.3, 4.01)
- moved C14 1.53 mm to (29.6, 3.05), turned to 180 degrees
- moved R7 0.57 mm to (21.3, 5.33), flipped to the bottom, turned to 180 degrees
- moved C3 0.08 mm to (31.8, 9.32)
Routing:
- net 3V3: track 70.4 -> 77.0 mm, vias 7 -> 8
- net GND: track 12.8 -> 18.3 mm
- net N$17: track 9.69 -> 5.28 mm
- net DVDD_1: track 12.9 -> 8.94 mm
- net PHASE_A1: track 28.4 -> 31.1 mm
- net NRST: track 31.6 -> 29.2 mm
- net FAULT_1: track 23.5 -> 24.9 mm, vias 2 -> 0
- net INL_1: track 12.1 -> 10.7 mm, vias 2 -> 0
- net SLA_1: track 16.4 -> 15.0 mm
- net PHASE_B1: track 24.1 -> 25.4 mm
- net GLB_1: track 14.3 -> 15.5 mm
- net INHC_1: track 12.4 -> 11.6 mm
- net SLB_1: track 22.3 -> 21.6 mm
- net INHB_1: track 13.0 -> 12.3 mm
- net EN_1: track 15.9 -> 15.4 mm, vias 2 -> 0
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
Commit message: done
Parts:
- moved C11 1.02 mm to (47.4, 21.7)
- moved C39 1.02 mm to (37.1, 11.7)
- moved R3 1.02 mm to (47.4, 20.0)
- moved R5 1.02 mm to (47.4, 18.3)
- moved U$6 1.02 mm to (51.8, 10.2)
- moved U1 1.02 mm to (40.4, 10.9)
- moved C10 1.02 mm to (44.2, 20.8)
- moved C12 1.02 mm to (38.8, 11.6)
- moved C16 1.02 mm to (38.1, 14.2)
- moved C32 1.02 mm to (38.1, 8.99)
- moved C33 1.02 mm to (38.1, 7.19)
- moved C34 1.02 mm to (42.1, 7.26)
- moved C35 1.02 mm to (42.1, 8.97)
- moved C38 1.02 mm to (40.6, 11.6)
- moved C4 1.02 mm to (42.3, 11.6)
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Routing:
- net INL_1: track 10.7 -> 15.4 mm
- net 3V3: track 77.0 -> 74.7 mm
- net NRST: track 29.2 -> 28.2 mm
- net N$5: track 16.5 -> 15.5 mm
- net INHB_1: track 12.3 -> 13.4 mm
- net FAULT_1: track 24.9 -> 25.9 mm
- net EN_1: track 15.4 -> 16.4 mm
- net INHA_1: track 12.7 -> 13.7 mm
- net INHC_1: track 11.6 -> 12.6 mm
- net SWCLK: track 16.5 -> 15.5 mm
- net CAN_H: track 9.10 -> 8.08 mm
- net N$8: track 8.24 -> 7.22 mm
- net CAN_L: track 8.94 -> 7.92 mm
